Commit message: Implementation of CPG controller for trotting gait (symmetric)

File: assembly/Assem1.SLDASM/urdf/Assem1.SLDASM.urdf (robot description, URDF)
Before this commit: robot Assem1.SLDASM, 9 links, 8 joints
Joints:
- joint bll: limit lower=0 upper=0 effort=0 velocity=0 -> lower=-1.57 upper=1.57 effort=500 velocity=10
- joint blu: limit lower=0 upper=0 effort=0 velocity=0 -> lower=-1.57 upper=1.57 effort=500 velocity=10
- joint brl: limit lower=0 upper=0 effort=0 velocity=0 -> lower=-1.57 upper=1.57 effort=500 velocity=10
- joint bru: limit lower=0 upper=0 effort=0 velocity=0 -> lower=-1.57 upper=1.57 effort=500 velocity=10
- joint fll: limit lower=0 upper=0 effort=0 velocity=0 -> lower=-1.57 upper=1.57 effort=500 velocity=10
- joint flu: limit lower=0 upper=0 effort=0 velocity=0 -> lower=-1.57 upper=1.57 effort=500 velocity=10
- joint frl: limit lower=0 upper=0 effort=0 velocity=0 -> lower=-1.57 upper=1.57 effort=500 velocity=10
- joint fru: limit lower=0 upper=0 effort=0 velocity=0 -> lower=-1.57 upper=1.57 effort=500 velocity=10
