Commit message: Changed URDF file, fixed reward function

File: assembly/Assem1_v3.SLDASM/urdf/Assem1_v3.SLDASM.urdf (robot description, URDF)
Before this commit: robot Assem1.SLDASM, 9 links, 8 joints
Links:
- link base_link: geometry collision mesh filename=package://Assem1_v3.SLDASM/meshes/base_link.STL; visual mesh filename=package://Assem1_v3.SLDASM/meshes/base_link.STL
- link bll_link: geometry collision mesh filename=package://Assem1_v3.SLDASM/meshes/bll_link.STL; visual mesh filename=package://Assem1_v3.SLDASM/meshes/bll_link.STL
- link blu_link: geometry collision mesh filename=package://Assem1_v3.SLDASM/meshes/blu_link.STL; visual mesh filename=package://Assem1_v3.SLDASM/meshes/blu_link.STL
- link brl_link: geometry collision mesh filename=package://Assem1_v3.SLDASM/meshes/brl_link.STL; visual mesh filename=package://Assem1_v3.SLDASM/meshes/brl_link.STL
- link bru_link: geometry collision mesh filename=package://Assem1_v3.SLDASM/meshes/bru_link.STL; visual mesh filename=package://Assem1_v3.SLDASM/meshes/bru_link.STL
- link fll_link: geometry collision mesh filename=package://Assem1_v3.SLDASM/meshes/fll_link.STL; visual mesh filename=package://Assem1_v3.SLDASM/meshes/fll_link.STL
- link flu_link: geometry collision mesh filename=package://Assem1_v3.SLDASM/meshes/flu_link.STL; visual mesh filename=package://Assem1_v3.SLDASM/meshes/flu_link.STL
- link frl_link: geometry collision mesh filename=package://Assem1_v3.SLDASM/meshes/frl_link.STL; visual mesh filename=package://Assem1_v3.SLDASM/meshes/frl_link.STL
- link fru_link: geometry collision mesh filename=package://Assem1_v3.SLDASM/meshes/fru_link.STL; visual mesh filename=package://Assem1_v3.SLDASM/meshes/fru_link.STL
Joints:
- joint bll: limit lower=-1.57 upper=1.57 effort=500 velocity=10 -> lower=-1.57 upper=1.57 effort=100 velocity=10; origin xyz=0.25 0 0 rpy=0 0 1.1163 -> xyz=0.25 0 0 rpy=0 0 1.11630563742211
- joint blu: limit lower=-1.57 upper=1.57 effort=500 velocity=10 -> lower=-1.57 upper=1.57 effort=100 velocity=10; origin xyz=0.79 -0.0225 0.055 rpy=-1.5708 1.3087 -3.1416 -> xyz=0.29 -0.055 0.2225 rpy=0 0 -1.83292456259005
- joint brl: limit lower=-1.57 upper=1.57 effort=500 velocity=10 -> lower=-1.57 upper=1.57 effort=100 velocity=10; origin xyz=0.25 0 0 rpy=0 0 -0.7862 -> xyz=0.25 0 0 rpy=0 0 -0.786196210632788
- joint bru: limit lower=-1.57 upper=1.57 effort=500 velocity=10 -> lower=-1.57 upper=1.57 effort=100 velocity=10; origin xyz=0.79 0.4225 0.055 rpy=-1.5708 1.5014 0 -> xyz=0.29 -0.055 -0.2225 rpy=3.14159265358979 0 -1.50135697543811
- joint fll: limit lower=-1.57 upper=1.57 effort=500 velocity=10 -> lower=-1.57 upper=1.57 effort=100 velocity=10; origin xyz=0.25 0 0 rpy=0 0 -1.1385 -> xyz=0.25 0 0 rpy=0 0 -1.13851717439948
- joint flu: limit lower=-1.57 upper=1.57 effort=500 velocity=10 -> lower=-1.57 upper=1.57 effort=100 velocity=10; origin xyz=0.21 -0.0225 0.055 rpy=1.5708 1.1212 0 -> xyz=-0.29 -0.0550000000000003 0.2225 rpy=0 0 -1.12122873429267
- joint frl: limit lower=-1.57 upper=1.57 effort=500 velocity=10 -> lower=-1.57 upper=1.57 effort=100 velocity=10; origin xyz=0.25 0 0 rpy=0 0 0.92792 -> xyz=0.25 0 0 rpy=0 0 0.927916437805553
- joint fru: limit lower=-1.57 upper=1.57 effort=500 velocity=10 -> lower=-1.57 upper=1.57 effort=100 velocity=10; origin xyz=0.21 0.4225 0.055 rpy=-1.5708 1.0032 0 -> xyz=-0.289999999999999 -0.0550000000000002 -0.2225 rpy=3.14159265358979 0 -1.00317652384274
