Commit message: Re-update local test files.

File: assembly/Assem1_v5.SLDASM/urdf/Assem1_v5.SLDASM.urdf (robot description, URDF)
Before this commit: robot Assem1_v5.SLDASM, 9 links, 8 joints
Joints:
- joint bll: limit lower=-0.785 upper=1.57 effort=100 velocity=50 -> lower=0.785 upper=-1.57 effort=100 velocity=50
- joint blu: limit lower=-0.785 upper=1.57 effort=100 velocity=50 -> lower=0.785 upper=-1.57 effort=100 velocity=50
- joint brl: axis 0 0 -1 -> 0 0 1; limit lower=-0.785 upper=1.57 effort=100 velocity=50 -> lower=0.785 upper=-1.57 effort=100 velocity=50
- joint bru: axis 0 0 -1 -> 0 0 1; limit lower=-0.785 upper=1.57 effort=100 velocity=50 -> lower=0.785 upper=-1.57 effort=100 velocity=50
- joint fll: limit lower=-0.785 upper=1.57 effort=100 velocity=50 -> lower=0.785 upper=-1.57 effort=100 velocity=50
- joint flu: limit lower=-0.785 upper=1.57 effort=100 velocity=50 -> lower=0.785 upper=-1.57 effort=100 velocity=50
- joint frl: axis 0 0 -1 -> 0 0 1; limit lower=-0.785 upper=1.57 effort=100 velocity=50 -> lower=0.785 upper=-1.57 effort=100 velocity=50
- joint fru: axis 0 0 -1 -> 0 0 1; limit lower=-0.785 upper=1.57 effort=100 velocity=50 -> lower=0.785 upper=-1.57 effort=100 velocity=50

Commit message: inital commit for 4 joints

File: assembly/Assem1_v5.SLDASM/urdf/Assem1_v5.SLDASM.urdf (robot description, URDF)
Before this commit: robot Assem1_v5.SLDASM, 9 links, 8 joints
Joints:
- joint bll: type revolute -> fixed
- joint brl: type revolute -> fixed
- joint fll: type revolute -> fixed
- joint frl: type revolute -> fixed
